File: kicad/current_version/working/working.kicad_pcb (KiCad board)
At the start: 2 copper layers, 201 parts, among them CON1 hi12pth

Commit message: commiting after auto generation
Parts:
- removed L198, L199, L200: l6r, oomlout_oomp_part_footprints:l6r_electronic_led_0603_red
- moved L174 203.2 mm to (-15.5, 241.3), turned to -58.1207 degrees
- moved L103 202.9 mm to (-19.8, 245.0), turned to -161.549 degrees
- moved L173 201.1 mm to (-13.9, 237.3), turned to -66.5112 degrees
- moved L175 199.6 mm to (-12.3, 242.0), turned to 45 degrees
- moved L172 199.0 mm to (-12.4, 233.4), turned to -66.5112 degrees
- moved L104 197.5 mm to (-18.7, 241.1), turned to 113.484 degrees
- moved L171 196.9 mm to (-10.8, 229.4), turned to -66.5112 degrees
- moved L176 194.7 mm to (-8.06, 242.0), turned to 45 degrees
- moved L105 191.3 mm to (-17.0, 236.8), turned to 113.484 degrees
- moved L177 189.8 mm to (-3.97, 241.8), turned to 88.9313 degrees
- moved L106 185.3 mm to (-15.3, 232.6), turned to 113.484 degrees
- moved L178 184.2 mm to (-2.41, 237.8), turned to 113.498 degrees
- moved L107 179.3 mm to (-13.6, 228.3), turned to 113.484 degrees
- moved L179 178.6 mm to (-0.85, 233.8), turned to 113.498 degrees
- moved L108 173.4 mm to (-11.9, 224.0), turned to 113.484 degrees
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